File: pcb/pcb.kicad_sch (KiCad schematic)
At the start: 206 parts, among them K0 Esc, K1 F1, K10 F10, K100 ., K11 F11, K12 F12, K13 PrtSc, K14 Del, K15 End, K16 PgUp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

Commit message: update pcb
Parts:
- K50: footprint Button_Switch_Keyboard:SW_Cherry_MX_1.25u_PCB -> Button_Switch_Keyboard:SW_Cherry_MX_ISOEnter_PCB
Other:
- moved on the sheet: D0, D1, D10, D100, D11, D12, D13, D14, D15, D16, D17, D18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
